File: FlightController/FlightController.kicad_pcb (KiCad board)
At the start: 2 copper layers, 55 x 55 mm, 51 parts, among them J1 USB_C_Receptacle_USB2.0_16P, J2 Conn_01x05, U1 ESP32-S3-WROOM-1, U2 AP2112K-3.3, U3 TVS0500DRV, U4 MCP6001R, U5 MS5611-01BA

Commit message: Add files via upload
Parts:
- removed the REF** at (156.0, 131.5)
- removed the REF** at (108.0, 83.5)
- removed the REF** at (108.0, 131.0)
- removed the REF** at (156.0, 83.5)
- removed TP1, TP2, TP3, TP4, TP5: TestPoint, TestPoint:TestPoint_Pad_2.0x2.0mm
- removed U1: ESP32-S3-WROOM-1, RF_Module:ESP32-S3-WROOM-1
- added J3: Conn_01x08, Connector_JST:JST_SHL_SM08B-SHLS-TF_1x08-1MP_P1.00mm_Horizontal, F.Cu at (169.6, 70.1)
- added REF**: MountingHole_4.5mm, MountingHole:MountingHole_4.5mm, F.Cu at (130.0, 80.0)
- added REF**: MountingHole_4.5mm, MountingHole:MountingHole_4.5mm, F.Cu at (100.0, 110.0)
- added REF**: MountingHole_4.5mm, MountingHole:MountingHole_4.5mm, F.Cu at (100.0, 80.0)
- added REF**: MountingHole_4.5mm, MountingHole:MountingHole_4.5mm, F.Cu at (130.0, 110.0)
- added U6: USBLC6-2SC6, Package_TO_SOT_SMD:SOT-23-6, F.Cu at (105.7, 97.6)
- added U7: ESP32-S3-MINI-1U, RF_Module:ESP32-S2-MINI-1U, F.Cu at (116.0, 94.2)
- J1: footprint Connector_USB:USB_C_Receptacle_GCT_USB4085 -> Connector_USB:USB_C_Receptacle_GCT_USB4110
- moved R4 126.0 mm to (65.4, 96.8)
- moved R3 125.7 mm to (65.4, 95.5)
- moved U3 124.9 mm to (81.6, 64.8)
- moved D1 117.9 mm to (65.6, 92.0), turned to -90 degrees
- moved F1 117.2 mm to (73.0, 88.7)
- moved C5 109.0 mm to (116.6, 82.1), turned to 90 degrees
- moved C4 108.6 mm to (117.8, 82.1), turned to 90 degrees
- moved C8 107.3 mm to (120.5, 84.6), turned to 180 degrees
- moved C9 106.4 mm to (120.5, 85.6), turned to 180 degrees
- moved C7 104.8 mm to (123.7, 82.4), turned to -90 degrees
- moved J2 104.7 mm to (148.1, 71.0)
- moved C6 102.7 mm to (124.9, 82.4), turned to -90 degrees
- moved R18 94.6 mm to (115.4, 82.1), turned to -90 degrees
- moved R1 87.6 mm to (158.5, 51.5)
- moved R11 87.6 mm to (161.4, 57.5)
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Connections:
- net /Raíz/D+ renamed Net-(J1-D+-PadA6)
- net /Raíz/D- renamed Net-(J1-D--PadA7)
- R6 pad 1: Net-(U1-IO38) -> /Raíz/M4_R
- R8 pad 1: Net-(U1-IO21) -> /Raíz/M3_R
Routing:
- net GND: track 0.00 -> 40.5 mm
- net /Raíz/3V3: track 0.00 -> 9.10 mm
- net /Raíz/5V: track 0.00 -> 5.85 mm
- net /Raíz/D+: track 0.00 -> 5.19 mm
- net /Raíz/D-: track 0.00 -> 3.71 mm
- net Net-(J1-D--PadA7): track 0.00 -> 2.69 mm
- net Net-(J1-D+-PadA6): track 0.00 -> 2.52 mm
- removed copper zone on B.Cu, net (none)
Other:
- board outline removed

Commit message: Add files via upload
Parts:
- added U1: MPU-6500, MisComponentes:MPU6500, F.Cu at (92.5, 55.3)
- moved C6 65.3 mm to (59.8, 87.7), turned to 90 degrees
- moved U2 63.6 mm to (57.2, 87.7)
- moved C4 63.6 mm to (54.5, 87.7)
- moved C5 63.4 mm to (53.4, 87.7)
- moved R18 63.2 mm to (52.4, 87.7)
- moved C7 62.9 mm to (61.0, 87.8), turned to 90 degrees
- moved J1 47.5 mm to (56.3, 76.8)
- moved U6 45.5 mm to (64.7, 77.8)
- moved R3 20.0 mm to (62.1, 75.7)
- moved U3 18.9 mm to (64.4, 72.7), turned to -90 degrees
- moved F1 18.8 mm to (62.1, 73.4), turned to -90 degrees
- moved R4 17.9 mm to (61.6, 79.3), turned to -90 degrees
- moved D1 17.2 mm to (68.2, 75.0), turned to 180 degrees
- moved C8 16.8 mm to (104.3, 89.1)
- moved C9 16.8 mm to (104.3, 90.1)
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Routing:
- net GND: track 40.5 -> 0.77 mm
- net /Raíz/3V3: track 9.10 -> 0.07 mm
- net /Raíz/5V: track 5.85 -> 0.03 mm
- net /Raíz/D+: track 5.19 -> 0.00 mm
- net /Raíz/D-: track 3.71 -> 0.00 mm
- net Net-(J1-D--PadA7): track 2.69 -> 0.00 mm
- net Net-(J1-D+-PadA6): track 2.52 -> 0.00 mm

Commit message: ACT
Parts:
- added C13: 100nF, Capacitor_SMD:C_0402_1005Metric, F.Cu at (120.6, 110.2)
- added C14: 100nF, Capacitor_SMD:C_0402_1005Metric, F.Cu at (116.9, 106.3)
- added J4: Conn_01x03, Connector_JST:JST_EH_B3B-EH-A_1x03_P2.50mm_Vertical, F.Cu at (96.1, 118.4)
- C1: value 0.1uF -> 10nF
- C3: value 0.1uF -> 100nF
- moved C10 107.3 mm to (100.2, 121.3)
- moved C11 105.5 mm to (104.0, 125.2), turned to -90 degrees
- moved U4 99.2 mm to (100.8, 125.1), turned to 90 degrees
- moved R15 98.3 mm to (102.2, 127.8), turned to 180 degrees
- moved R16 93.3 mm to (101.2, 122.3)
- moved R17 92.8 mm to (103.1, 125.2), turned to 90 degrees
- moved R14 88.8 mm to (101.7, 129.2), turned to 90 degrees
- moved C12 86.7 mm to (122.3, 119.5)
- moved R18 84.6 mm to (124.9, 131.2), turned to 0 degrees
- moved C5 83.1 mm to (124.9, 130.2), turned to 180 degrees
- moved C1 82.3 mm to (116.9, 107.3), turned to 180 degrees
- moved C4 81.7 mm to (124.9, 129.2), turned to 180 degrees
- moved C2 80.8 mm to (121.1, 111.8), turned to -90 degrees
- moved C3 80.2 mm to (120.2, 111.8), turned to 90 degrees
- moved U2 78.0 mm to (124.8, 126.5), turned to -90 degrees
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Connections:
- C1 pad 1: Net-(MPU1-VDD) -> Net-(U1-VDD)
- C2 pad 1: Net-(MPU1-VDDIO) -> /Raíz/VDDIO
- C3 pad 2: Net-(MPU1-FSYNC) -> /Raíz/VDDIO
- R1 pad 2: /Raíz/SCL -> Net-(U1-SCL/SCLK)
- R2 pad 2: /Raíz/SDA -> Net-(U1-SDA/SDI)
- U1 pad 10: unconnected-(U1-REGOUT-Pad10) -> Net-(U1-REGOUT)
- U1 pad 11: unconnected-(U1-FSYNC-Pad11) -> GND
- U1 pad 12: unconnected-(U1-INT-Pad12) -> /Raíz/INT
- U1 pad 13: unconnected-(U1-VDD-Pad13) -> Net-(U1-VDD)
- U1 pad 18: unconnected-(U1-GND-Pad18) -> GND
- U1 pad 22: unconnected-(U1-NCS-Pad22) -> /Raíz/3V3
- U1 pad 23: unconnected-(U1-SCL/SCLK-Pad23) -> Net-(U1-SCL/SCLK)
- U1 pad 24: unconnected-(U1-SDA/SDI-Pad24) -> Net-(U1-SDA/SDI)
- U1 pad 25: unconnected-(U1-EXP-Pad25) -> GND
- U1 pad 7: unconnected-(U1-AUX_CL-Pad7) -> GND
- U1 pad 8: unconnected-(U1-VDDIO-Pad8) -> /Raíz/VDDIO
- U1 pad 9: unconnected-(U1-AD0/SDO-Pad9) -> GND
- U7 pad 19: /Raíz/M2_R -> /Raíz/M1_R
- U7 pad 20: /Raíz/M1_R -> /Raíz/M2_R

Commit message: Add files via upload
Parts:
- removed R10, R11, R12, R13, R6, R7, R8, R9: R_Small, Resistor_SMD:R_0402_1005Metric
- J2: footprint Connector_JST:JST_EH_B5B-EH-A_1x05_P2.50mm_Vertical -> Connector_PinHeader_2.54mm:PinHeader_1x05_P2.54mm_Vertical
- J4: footprint Connector_JST:JST_EH_B3B-EH-A_1x03_P2.50mm_Vertical -> Connector_PinHeader_2.54mm:PinHeader_1x03_P2.54mm_Vertical
- moved U5 34.6 mm to (101.6, 88.6)
- moved R20 34.6 mm to (102.7, 91.0)
- moved C12 34.6 mm to (101.1, 92.1)
- moved R19 34.6 mm to (100.4, 91.0)
- moved C4 33.2 mm to (127.5, 96.1)
- moved C5 33.2 mm to (127.5, 97.1)
- moved C6 33.2 mm to (127.5, 90.7)
- moved C7 33.2 mm to (127.5, 89.5)
- moved R18 33.2 mm to (127.5, 98.1)
- moved U2 33.2 mm to (127.4, 93.3)
- moved R14 32.4 mm to (105.5, 97.1), turned to 180 degrees
- moved R15 31.2 mm to (104.0, 96.6), turned to -90 degrees
- moved C11 30.6 mm to (101.5, 94.7), turned to 0 degrees
- moved R17 29.5 mm to (101.5, 95.7), turned to 180 degrees
- moved U4 27.1 mm to (101.4, 98.0), turned to 180 degrees
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Connections:
- J3 pad 3: /Raíz/M4 -> /Raíz/M4_R
- J3 pad 4: /Raíz/M3 -> /Raíz/M3_R
- J3 pad 5: /Raíz/M2 -> /Raíz/M2_R
- J3 pad 6: /Raíz/M1 -> /Raíz/M1_R
