File: FlightController/FlightController.kicad_sch (KiCad schematic)
At the start: 41 parts, among them J1 USB_C_Receptacle_USB2.0_16P, J2 Conn_01x05, U1 ESP32-S3-WROOM-1, U2 AP2112K-3.3, U3 TVS0500DRV, U4 ${SIM.PARAMS}

Commit message: Add files via upload
Parts:
- removed MS3: (no value), symbol MisComponentes:HB100
- removed U4: ${SIM.PARAMS}, symbol Simulation_SPICE:OPAMP
Connections:
- net GPIO1: now reaches U1.39 (IO1)
Changed lines of the file:
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@@
 	(wire
 		(pts
+			(xy 143.51 46.99) (xy 146.05 46.99)
+		)
+		(stroke
+			(width 0)
+			(type default)
+		)
+	)
+	(wire
+		(pts
 			(xy 184.15 114.3) (xy 189.23 114.3)
 		)
@@
 		)
 	)
+	(label "GPIO1"
+		(at 143.51 46.99 180)
+		(effects
+			(font
+				(size 1.27 1.27)
+			)
+			(justify right bottom)
+		)
+	)
 	(label "3V3"
 		(at 44.45 27.94 90)
@@
 		)
 	)
-	(label "OPAMP - TLV2462"
-		(at 67.31 160.02 0)
-		(effects
-			(font
-				(size 1.27 1.27)
-				(thickness 0.254)
-				(bold yes)
-			)
-			(justify left bottom)
-		)
-	)
 	(label "M2"
 		(at 128.27 119.38 90)
@@
 	)
 	(symbol
-		(lib_id "MisComponentes:HB100")
-		(at 110.49 187.96 0)
-		(unit 1)
-		(body_style 1)
-		(exclude_from_sim no)
-		(in_bom yes)
-		(on_board yes)
-		(in_pos_files yes)
-		(dnp no)
-		(fields_autoplaced yes)
-		(property "Reference" "MS3"
-			(at 116.84 185.4199 0)
-			(show_name no)
-			(do_not_autoplace no)
-			(effects
-				(font
-					(size 1.27 1.27)
-				)
-				(justify left)
-			)
-		)
-		(property "Value" ""
-			(at 110.49 187.96 0)
-			(show_name no)
-			(do_not_autoplace no)
-			(effects
-				(font
-					(size 1.27 1.27)
-				)
-			)
-		)
-		(property "Footprint" ""
-			(at 110.49 187.96 0)
-			(hide yes)
-			(show_name no)
-			(do_not_autoplace no)
-			(effects
-				(font
-					(size 1.27 1.27)
-				)
-			)
-		)
-		(property "Datasheet" ""
-			(at 110.49 187.96 0)
-			(hide yes)
-			(show_name no)
-			(do_not_autoplace no)
-			(effects
-				(font
-					(size 1.27 1.27)
-				)
-			)
-		)
-		(property "Description" ""
-			(at 110.49 187.96 0)
-			(hide yes)
-			(show_name no)
-			(do_not_autoplace no)
-			(effects
-				(font
-					(size 1.27 1.27)
-				)
-			)
-		)
-		(pin ""
-		)
-		(pin ""
-		)
-		(pin ""
-		)
-		(pin ""
-		)
-		(instances
-			(project "FlightController"
-				(path "/308dac0f-86ec-4e6d-81af-c05338252f11"
-					(reference "MS3")
-					(unit 1)
-				)
-			)
-		)
-	)
-	(symbol
 		(lib_id "power:Earth")
 		(at 49.53 31.75 180)
@@
 					(unit 1)
 				)
-			)
-		)
-	)
-	(symbol
-		(lib_id "Simulation_SPICE:OPAMP")
-		(at 81.28 185.42 0)
-		(unit 1)
-		(body_style 1)
-		(exclude_from_sim no)
-		(in_bom yes)
-		(on_board yes)
-		(in_pos_files yes)
-		(dnp no)
-		(fields_autoplaced yes)
-		(property "Reference" "U4"
-			(at 88.9 180.2698 0)
-			(show_name no)
-			(do_not_autoplace no)
-			(effects
-				(font
-					(size 1.27 1.27)
-				)
-			)
-		)
-		(property "Value" "${SIM.PARAMS}"
-			(at 88.9 182.1749 0)
-			(show_name no)
-			(do_not_autoplace no)
-			(effects
-				(font
-					(size 1.27 1.27)
-				)
-			)
-		)
-		(property "Footprint" ""
-			(at 81.28 185.42 0)
-			(hide yes)
-			(show_name no)
-			(do_not_autoplace no)
-			(effects
-				(font
-					(size 1.27 1.27)
-				)
-			)
-		)
-		(property "Datasheet" "https://ngspice.sourceforge.io/docs/ngspice-html-manual/manual.xhtml#sec__SUBCKT_Subcircuits"
-			(at 81.28 185.42 0)
-			(hide yes)
-			(show_name no)
-			(do_not_autoplace no)
-			(effects
-				(font
-					(size 1.27 1.27)
-				)
-			)
-		)
-		(property "Description" "Operational amplifier, single"
-			(at 81.28 185.42 0)
-			(hide yes)
-			(show_name no)
-			(do_not_autoplace no)
-			(effects
-				(font
-					(size 1.27 1.27)
-				)
-			)
-		)
-		(property "Sim.Pins" "1=in+ 2=in- 3=vcc 4=vee 5=out"
-			(at 81.28 185.42 0)
-			(hide yes)
-			(show_name no)
-			(do_not_autoplace no)
-			(effects
-				(font
-					(size 1.27 1.27)
-				)
-			)
-		)
-		(property "Sim.Device" "SUBCKT"
-			(at 81.28 185.42 0)
-			(hide yes)
-			(show_name no)
-			(do_not_autoplace no)
-			(effects
-				(font
-					(size 1.27 1.27)
-				)
-				(justify left)
-			)
-		)
-		(property "Sim.Library" "${KICAD9_SYMBOL_DIR}/Simulation_SPICE.sp"
-			(at 81.28 185.42 0)
-			(hide yes)
-			(show_name no)
-			(do_not_autoplace no)
-			(effects
-				(font
-					(size 1.27 1.27)
-				)
-			)
-		)
-		(property "Sim.Name" "kicad_builtin_opamp"
-			(at 81.28 185.42 0)
-			(hide yes)
-			(show_name no)
-			(do_not_autoplace no)
-			(effects
-				(font
-					(size 1.27 1.27)
-				)
-			)
-		)
-		(pin "3"
-		)
-		(pin "4"
-		)
-		(pin "5"
-		)
-		(pin "1"
-		)
-		(pin "2"
-		)
-		(instances
-			(project "FlightController"
-				(path "/308dac0f-86ec-4e6d-81af-c05338252f11"
-					(reference "U4")
-					(unit 1)
-				)

Commit message: Add files via upload
Parts:
- removed MS1: (no value), symbol MisComponentes:MS5611
- added C12: 0.1uF, Capacitor_SMD:C_0402_1005Metric, symbol Device:C
- added R18: 5.1K, Resistor_SMD:R_0402_1005Metric, symbol Device:R_US
- added R19, R20: 1K, symbol Device:R
- added U5: MS5611-01BA, Package_LGA:LGA-8_3x5mm_P1.25mm, symbol Sensor_Pressure:MS5611-01BA
- C1, C2, C3, C4, C5, C6, C7, C8, C9: footprint (none) -> Capacitor_SMD:C_0402_1005Metric
- D1, D2: footprint (none) -> Diode_SMD:D_SOD-123
- F1: footprint (none) -> Fuse:Fuse_0805_2012Metric
- J1: footprint (none) -> Connector_USB:USB_C_Receptacle_GCT_USB4085
- J2: footprint (none) -> Connector_JST:JST_EH_B5B-EH-A_1x05_P2.50mm_Vertical
- R1, R10, R11, R12, R13, R2, R3, R4, R5, R6, R7, R8, R9: footprint (none) -> Resistor_SMD:R_0402_1005Metric
- TP1, TP2, TP3, TP4, TP5: footprint (none) -> TestPoint:TestPoint_Pad_2.0x2.0mm
Connections:
- net GND: now also U3.1 (GND), U3.2 (GND), U3.3 (GND), U3.7 (GND), C12.2, R18.1, R20.2, U5.3 (GND); no longer U3.4 (IN), U3.5 (IN), U3.6 (IN)
- net SCL: now also U5.8 (SCLK)
- net SDA: now also U5.7 (SDI/SDA)
- net +3V3 renamed 3V3
- net 3V3: now also C12.1, R18.2, R19.1, U5.1 (VDD)
- net +5V renamed 5V
- removed net S: D1.2 (A), U3.1 (GND), U3.2 (GND), U3.3 (GND), U3.7 (GND)
- new net: D1.2 (A), U3.4 (IN), U3.5 (IN), U3.6 (IN)
- new net: R19.2, U5.2 (PS)
- new net: R20.1, U5.4 (CSB), U5.5 (CSB)
- no-connect marks 12 -> 44
Other:
- note removed: "CONTROL"
- note removed: "Capacitors must be placed the nearest possible to the pin on the PCB"
- note removed: "MCU"
- note removed: "POTENCIA"
- note removed: "R6, R8, R10, R12 → 33Ω R7, R9, R11, R13 → 10k"
- moved on the sheet: C4, C5, C6, C7, D1, U2, U3

Commit message: Add files via upload
Parts:
- removed TP1, TP2, TP3, TP4, TP5: TestPoint, TestPoint:TestPoint_Pad_2.0x2.0mm, symbol Connector:TestPoint
- added J3: Conn_01x08, symbol Connector_Generic:Conn_01x08
- R19, R20: footprint (none) -> Resistor_SMD:R_0402_1005Metric
Connections:
- net GND: now also J3.8 (Pin_8)
- net M1: now also J3.6 (Pin_6)
- net M2: now also J3.5 (Pin_5)
- net M3: now also J3.4 (Pin_4)
- net M4: now also J3.3 (Pin_3)
- new net C: J3.2 (Pin_2)
- no-connect marks 44 -> 46

Commit message: Add files via upload
Parts:
- removed U1: ESP32-S3-WROOM-1, RF_Module:ESP32-S3-WROOM-1, symbol RF_Module:ESP32-S3-WROOM-1
- added U6: USBLC6-2SC6, Package_TO_SOT_SMD:SOT-23-6, symbol Power_Protection:USBLC6-2SC6
- added U7: ESP32-S3-MINI-1U, RF_Module:ESP32-S2-MINI-1U, symbol RF_Module:ESP32-S3-MINI-1U
- J1: footprint Connector_USB:USB_C_Receptacle_GCT_USB4085 -> Connector_USB:USB_C_Receptacle_GCT_USB4110
- J3: footprint (none) -> Connector_JST:JST_SHL_SM08B-SHLS-TF_1x08-1MP_P1.00mm_Horizontal
Connections:
- net 3V3: now also U7.3 (3V3)
- net D+: now also U6.4 (I/O2), U7.24 (USB_D+); no longer J1.A6 (D+), J1.B6 (D+)
- net D-: now also U6.6 (I/O1), U7.23 (USB_D-); no longer J1.A7 (D-), J1.B7 (D-)
- net GND: now also U6.2 (GND), U7.1 (GND), U7.2 (GND), U7.42 (GND), U7.43 (GND), U7.46 (GND), U7.47 (GND), U7.48 (GND), U7.49 (GND), U7.50 (GND), U7.51 (GND), U7.52 (GND), U7.53 (GND), U7.54 (GND), U7.55 (GND), U7.56 (GND), U7.57 (GND), U7.58 (GND), U7.59 (GND), U7.60 (GND), U7.61 (GND), U7.62 (GND), U7.63 (GND), U7.64 (GND), U7.65 (GND)
- net GPIO1: now also U7.5 (IO1)
- net INT: now also U7.30 (IO48)
- net M1_R: now also U7.20 (IO16)
- net M2_R: now also U7.19 (IO15)
- net SCL: now also U7.31 (IO35)
- net SDA: now also U7.32 (IO36)
- net M3_R: now reaches R8.1
- net M3_R: now also U7.21 (IO17)
- net M4_R: now reaches R6.1
- net M4_R: now also U7.22 (IO18)
- new net: J1.A6 (D+), J1.B6 (D+), U6.3 (I/O2)
- new net: J1.A7 (D-), J1.B7 (D-), U6.1 (I/O1)
- no-connect marks 46 -> 47
Other:
- moved on the sheet: C8, C9, R6, R7, R8, R9

Commit message: Add files via upload
Parts:
- added U1: MPU-6500, MisComponentes:MPU6500, symbol MisComponentes:MPU-6500

Commit message: ACT
Parts:
- removed MPU1: (no value), symbol MisComponentes:MPU-6500FINAL
- added C13, C14: 100nF, Capacitor_SMD:C_0402_1005Metric, symbol Device:C
- C1: value 0.1uF -> 10nF
- C3: value 0.1uF -> 100nF
Connections:
- net 3V3: now also U1.22 (NCS)
- net GND: now also U1.11 (FSYNC), U1.18 (GND), U1.25 (EXP), U1.7 (AUX_CL), U1.9 (AD0/SDO), C13.1, C14.1
- net INT: now also U1.12 (INT)
- net M1_R: now also U7.19 (IO15); no longer U7.20 (IO16)
- net M2_R: now also U7.20 (IO16); no longer U7.19 (IO15)
- net SCL: no longer R1.2
- net SDA: no longer R2.2
- net VDDIO: now reaches C3.2
- net VDDIO: now also C2.1, U1.8 (VDDIO)
- net at C1.1: now also U1.13 (VDD), C14.2
- net at U1.10 (REGOUT): now also C13.2
- net at U1.23 (SCL/SCLK): now also R1.2
- net at U1.24 (SDA/SDI): now also R2.2
- no-connect marks 47 -> 37
Other:
- moved on the sheet: C1, C2, C3, R1, R2, R5, U1

Commit message: Add files via upload
Parts:
- removed R10, R11, R12, R13, R6, R7, R8, R9: R_Small, Resistor_SMD:R_0402_1005Metric, symbol Device:R_Small
- J2: footprint Connector_JST:JST_EH_B5B-EH-A_1x05_P2.50mm_Vertical -> Connector_PinHeader_2.54mm:PinHeader_1x05_P2.54mm_Vertical
Connections:
- net M1 is gone; now on net M1_R: J3.6 (Pin_6)
- net M2 is gone; now on net M2_R: J3.5 (Pin_5)
- net M3 is gone; now on net M3_R: J3.4 (Pin_4)
- net M4 is gone; now on net M4_R: J3.3 (Pin_3)
Other:
- note added: "FALTA PROBAR LAS SALIDAS DEL D_SHOT HACIA EL ESC PARA VER SI LO LEE A 3V3 PORQUE EL ESC NO ESPECIFICA EL VOLTAJE DE LECTURA"
- moved on the sheet: J2, J3
